File: ESP8266_1wire_Gateway/ESP8266_1wire_Gateway.sch (EAGLE design)
At the start: 70 parts, among them IC1 5V, IC2 3.3V, IC3 DS2482-100S, IC4 DS18B20, Q1 BSS84, Q2 BSS138, Q3 BSS138

Commit message: .
Parts:
- removed FLASH_SW: DTSM-3, mechanics:DTSM-3
Connections:
- net GND: no longer FLASH_SW.2
- net N$10: no longer FLASH_SW.1
Other:
- note removed: "mit SJ1 und SJ2 kann ESD-Schutz überbrückt werden (ZD1 entfällt) mit SJ4 und SJ3 kann BusMaster überbrückt werden und eine andere GPIO für 1W-Signal verwendet werden (I2C bleibt anderweitig benutzbar) (IC3, Q3, R14, R11 entfallen)"
- moved on the sheet: CLR, FLASH, I2C_1, I2C_2, IC4

Commit message: v0.9
Parts:
- removed CLR: (no value), my:PINHD-1X2_S
- removed G12, G13: LSP10, my:LSP10
- added 1W1, 1W2: (no value), my:PINHD-1X3_S
- added G4, G5: LSP10, my:LSP10
- added HSPI: (no value), my:PINHD-1X4_S
- RST: value GND -> RST
- renumbered GND8 to RST
Connections:
- net CSN renamed GPIO15
- removed net GPIO0: G0.MP, MDL1.GPIO0, R12.2, R5.1
- removed net GPIO2: G2.MP, MDL1.GPIO2, R4.1, SJ3.1
- new net 1WDIR: G0.MP, MDL1.GPIO0, R12.2, R5.1, SJ3.1
- new net GPIO5: G5.MP, MDL1.GPIO5, R8.1
- new net HCS0: HSPI.4, MDL1.CS0
- new net HMISO: HSPI.3, MDL1.MISO
- new net HMOSI: HSPI.2, MDL1.MOSI
- new net HSCLK: HSPI.1, MDL1.SCLK
- net 1W_ESD: now also 1W1.2, 1W2.2
- net GND: no longer RST.MP
- net GND_ESD: now also 1W1.3, 1W2.3
- net LED_OPT: now also G4.MP, MDL1.GPIO4, R9.1; no longer G12.MP, MDL1.GPIO12, R8.1
- net RST: now also RST.MP
- net RXD: no longer CLR.2
- net SCL1: now also MDL1.GPIO12; no longer MDL1.GPIO5
- net SDA1: now also MDL1.GPIO13; no longer MDL1.GPIO4
- net SW_OPT: now also G2.MP, MDL1.GPIO2, R4.1; no longer G13.MP, MDL1.GPIO13, R9.1
- net TXD: no longer CLR.1
- net VCC_5V: now also 1W1.1, 1W2.1
Other:
- moved on the sheet: IC4, R8, R9, SCL, SDA
