File: ESP8266_MySensorsGateway/ESP8266_MySensorsGateway_v1.3.sch (EAGLE design)
At the start: 73 parts, among them IC1 5V, IC2 3.3V, IC3 DS2482-100S, IC4 DS18B20, Q1 BSS84, Q2 BSS138, Q3 BSS138, Q4 BSS138

Commit message: Version 1.2 : ELKO / THT Version 1.3 : tantal / SMD
Parts:
- removed 1W: 1Wire, my:W237-03P
- removed 1W1, 1W2: (no value), my:PINHD-1X3_S
- removed 3V3, 5V, ADC, G0, G12, G13, G14, G15, G2, G4, G5, GND: LSP10, my:LSP10
- removed C6: 104, resistor:C-EUC0805
- removed C7: 100uF, rcl:CPOL-EUE2,5-6E
- removed C8: 470pF, resistor:C-EUC0805
- removed GND1: GND, my:LSP10
- removed HSPI, I2C_1, I2C_2: (no value), my:PINHD-1X4_S
- removed IC2: 3.3V, SparkFun-PowerIC:V_REG_LM1117SOT223
- removed IC3: DS2482-100S, my:DS2482-100S
- removed IC4: DS18B20, my:DS18B20
- removed JP1: USB-MICROB, SparkFun-Connectors:USB-MICROB
- removed LED1: CFG, led:LEDCHIPLED_1206
- removed MDL1: µC, ESP8266-ESP12E:ESP8266-12EESP8266-ESP12E
- removed OPT, RESET: DTSM-3, mechanics:DTSM-3
- removed Q1: BSS84, transistor-small-signal:BSS84
- removed Q2, Q3, Q4: BSS138, my:BSS138
- removed R16: 4k7, resistor:R-EU_R0805
- removed R17: 100, my:R0805_SMALL_GAP
- removed R18: ?, my:R0805_SMALL_GAP
- removed R19: 10k, rcl:R-EU_R0805
- removed R20: 470, resistor:R-EU_R0805
- removed R21, R22: 10k, resistor:R-EU_R0805
- removed VIN: 7-14, my:W237-02P
- removed X1: (no value), my:CON_350-104
- removed X3: (no value), my:CON_350-102
- removed ZD1, ZD2: DS9503_BYPASS_JP, my:DS9503_BYPASS_JP
- added ERR: R, led:LEDCHIPLED_1206
- added ESP: µC, ESP8266-ESP12E:ESP8266-12EESP8266-ESP12E
- added INCLUSION: DTSM-3, mechanics:DTSM-3
- added PWR: Vin, my:W237-02P
- added RADIO1: NRF24L01+, my:NRF24L01+
- added RADIO2: NRF24L01+NRF24L01+MINI, my:NRF24L01+NRF24L01+MINI
- added RX: G, led:LEDCHIPLED_1206
- added TX: Y, led:LEDCHIPLED_1206
- added USB: USB-MICROB, SparkFun-Connectors:USB-MICROB
- C1, C5: value 105 -> 104
- C2: value 104 -> 107; device resistor:C-EUC0805 -> my:C
- C3: value 0,1mF -> 105
- C4: value 100mF -> 104; device resistor:C-EUC1210 -> resistor:C-EUC0805
- FLASH: value (none) -> DTSM-3; device my:PINHD-1X2_S -> mechanics:DTSM-3
- IC1: value 5V -> 3V3
- PF1: value 500mA -> PTC-F1206
- PRG: value (none) -> (none)
- R10: value 220k -> 10k
- R11: value 100k -> 10k
- R12: value 470 -> 10k; device resistor:R-EU_R0805 -> rcl:R-EU_R0805
- R13, R14: value 4k7 -> 10k; device resistor:R-EU_R0805 -> rcl:R-EU_R0805
- R15: value 4k7 -> 470
- RST: value RST -> DTSM-3; device my:LSP10 -> mechanics:DTSM-3
- SJ1: value JUMPER-PAD-2-NOYES_SILK -> JUMPER-PAD-3-2OF3_NC_BY_TRACE_SMALL; device SparkFun-Passives:JUMPER-PAD-2-NOYES_SILK -> SparkFun-Passives:JUMPER-PAD-3-2OF3_NC_BY_TRACE_SMALL
Connections:
- removed net 1W: IC3.1W, R17.2
- removed net 1WDIR: G0.MP, MDL1.GPIO0, Q4.S, R12.2, R21.2, R5.1, SJ1.2
- removed net 1WD_ESD: ZD2.P$4
- removed net 1W_: Q1.D, R17.1, ZD1.P$1
- removed net 1W_1: Q4.D, R22.2, SJ1.1, ZD2.P$1
- removed net 1W_ESD: 1W-2.KL, 1W1.2, 1W2.2, IC4.1W, ZD1.P$4
- removed net 5V_IN: C2.1, IC1.OUT, JP1.VBUS, PF1.2
- removed net ADC: MDL1.ADC, R10.2, R11.2
- removed net GNDD_ESD: ZD2.P$3
- removed net GND_ESD: 1W-3.KL, 1W1.3, 1W2.3, IC4.GND, ZD1.P$3
- removed net GPIO13: G13.MP, MDL1.GPIO13
- removed net GPIO14: G14.MP, MDL1.GPIO14, R7.1
- removed net GPIO15: G15.MP, MDL1.GPIO15, R6.2
- removed net HCS0: HSPI.4, MDL1.CS0
- removed net HMISO: HSPI.3, MDL1.MISO
- removed net HMOSI: HSPI.2, MDL1.MOSI
- removed net HSCLK: HSPI.1, MDL1.SCLK
- removed net LED_OPT: G12.MP, MDL1.GPIO12, R19.1
- removed net N$11: OPT.1, R20.1
- removed net N$8: C1.1, D1.CATHODE, IC1.IN
- removed net SCL1: G5.MP, I2C_1.3, I2C_2.3, MDL1.GPIO5, Q3.S, R14.1, R8.1
- removed net SCL2: IC3.SCL, Q3.D, R16.1
- removed net SDA1: G4.MP, I2C_1.4, I2C_2.4, MDL1.GPIO4, Q2.S, R13.1, R9.1
- removed net SDA2: IC3.SDA, Q2.D, R15.1
- removed net SW_OPT: G2.MP, MDL1.GPIO2, R20.2, R4.1
- removed net VCC_5V: 1W-1.KL, 1W1.1, 1W2.1, 5V.MP, C5.1, IC2.IN, IC3.VDD, IC4.VDD, PF1.1, R15.2, R16.2, R18.2, R22.1
- new net CE: ESP.GPIO4, R11.1, RADIO1.CE, RADIO2.CE
- new net CSN: ESP.GPIO15, R6.2, RADIO1.CSN, RADIO2.CSN
- new net GPIO0: ESP.GPIO0, R15.2, R5.1
- new net INCL: ESP.GPIO5, INCLUSION.1, R10.1
- new net IRQ: RADIO1.IRQ, RADIO2.IRQ
- new net LED_ERR: ESP.GPIO2, R12.1, R4.1
- new net L_BASE: ERR.A, RX.A, SJ1.2, TX.A
- new net MISO: ESP.GPIO12, R8.1, RADIO1.MISO, RADIO2.MISO
- new net MOSI: ESP.GPIO13, R9.1, RADIO1.MOSI, RADIO2.MOSI
- new net SCK: ESP.GPIO14, R7.1, RADIO1.SCK, RADIO2.SCK
- new net VUSB: D1.CATHODE, PF1.1, USB.VBUS
- net CH_PD: now also ESP.CH_PD; no longer MDL1.CH_PD
- net DEEP_SLEEP: now also ESP.GPIO16; no longer MDL1.GPIO16
- net GND: now also ESP.GND, FLASH.2, INCLUSION.2, PWR-1.KL, RADIO1.GND, RADIO2.GND, RST.1, SJ1.1, USB.GND; no longer C6.2, C7.-, C8.2, FLASH.1, GND.MP, GND1.MP, I2C_1.2, I2C_2.2, IC2.ADJ, IC3.AD0, IC3.AD1, IC3.GND, JP1.GND, LED1.A, MDL1.GND, OPT.2, R11.1, RESET.1, VIN-1.KL, ZD1.P$2, ZD2.P$2
- net N$10: now also C3.1, IC1.IN, PF1.2; no longer FLASH.2, R12.1
- net N$4: now also ERR.C, R12.2; no longer LED1.C, R19.2
- net N$5: now also R13.2, TX.C; no longer ADC.MP, R10.1
- net N$6: now also R14.2, RX.C; no longer IC3.PCT, Q1.G
- net N$7: now also FLASH.1, R15.1; no longer Q1.S, R18.1
- net RST: now also ESP.REST, RST.2; no longer C8.1, MDL1.REST, RESET.2, RST.MP
- net RXD: now also ESP.RXD, R14.1; no longer MDL1.RXD
- net TXD: now also ESP.TXD, R13.1; no longer MDL1.TXD
- net VCC: now also C1.1, C2.1, C5.1, ESP.VCC, IC1.OUT, R10.2, R11.2, RADIO1.VCC, RADIO2.VCC, SJ1.3; no longer 3V3.MP, C3.1, C6.1, C7.+, I2C_1.1, I2C_2.1, IC2.OUT, MDL1.VCC, Q2.G, Q3.G, Q4.G, R13.2, R14.2, R21.1
- net VIN: now also PWR-2.KL; no longer VIN-2.KL
Other:
- note added: "5-14V"
- note added: "ESP MySensors Gateway"
- note added: "ESP8266 MySensors Gateway"
- note added: "Error (R)"
- note added: "LEDs"
- note added: "RX (G)"
- note added: "Radio"
- note added: "TX (Y)"
- note added: "deep sleep (ansonsten kann dieser Widerstand entfallen)"
- note added: "freie GPIOs"
- note added: "primäre Versorgung"
- note removed: "7-14V"
- note removed: "ESP 1wire Gateway"
- note removed: "ESP8266 1wire Gateway"
- note removed: "Opt"
- note removed: "WLAN-1wire Gateway Schaltungsbeschreibung: - basierend auf ESP8266 (ESP-12). - vorbereitet zum direkten Anschluss von 1wire-Devices (Schraubklemmen) - Bus1 mit Busmaster-Chip (IC3, DS2482-100S) - 1w-Bus-Versorgung mit 5V (MOSFET-LevelShifter Q2,Q3) - Bus2 direkt per GPIO0 - optionaler (überbrückbarer) LevelShifter (SJ1) für 5V-Versorgung - optionaler ESD-Schutz (ZD1, DS9503P), überbrückbar für Bu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"
- note removed: "current limiting resistor"
- note removed: "line termination resistor typically 100 Ohm"
- moved on the sheet: C1, C2, C3, C4, C5, D1, IC1, PF1, PRG, R1, R10, R11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

Commit message: version 1.3
Parts:
- USB: value USB-MICROB -> USB_MICROB_PLUGCONN-11752; device SparkFun-Connectors:USB-MICROB -> SparkFun-Connectors:USB_MICROB_PLUGCONN-11752
Connections:
- net GND: now also USB.SHIELD
- net VUSB: now also USB.VCC; no longer USB.VBUS
Changed lines of the file:
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@@
 <setting verticaltext="up"/>
 </settings>
-<grid distance="0.1" unitdist="inch" unit="inch" style="lines" multiple="1" display="no" altdistance="0.01" altunitdist="inch" altunit="inch"/>
+<grid distance="25" unitdist="mil" unit="mil" style="lines" multiple="1" display="no" altdistance="0.01" altunitdist="inch" altunit="inch"/>
 <layers>
 <layer number="1" name="Top" color="4" fill="1" visible="no" active="no"/>
@@
 <part name="SJ1" library="SparkFun-Passives" deviceset="JUMPER-PAD-3-2OF3_NC_BY_TRACE" device="_SMALL"/>
 <part name="GND3" library="supply1" deviceset="GND" device=""/>
-<part name="USB" library="SparkFun-Connectors" deviceset="USB" device="-MICROB"/>
 <part name="PRG" library="my" deviceset="PINHD-1X4_S" device=""/>
 <part name="C5" library="resistor" deviceset="C-EU" device="C0805" value="104"/>
 <part name="R15" library="resistor" deviceset="R-EU_" device="R0805" value="470"/>
 <part name="C2" library="my" deviceset="C" device="" value="107"/>
+<part name="USB" library="SparkFun-Connectors" deviceset="USB_MICROB_PLUG" device="CONN-11752"/>
 </parts>
 <sheets>
@@
 <instance part="SJ1" gate="G$1" x="-24.13" y="-17.78" smashed="yes" rot="MR180"/>
 <instance part="GND3" gate="1" x="-17.145" y="-22.86" rot="R90"/>
-<instance part="USB" gate="G$1" x="164.592" y="18.415"/>
 <instance part="PRG" gate="A" x="101.6" y="83.82"/>
 <instance part="C5" gate="G$1" x="132.08" y="73.66" smashed="yes" rot="R90">
@@
 <instance part="R15" gate="G$1" x="69.85" y="63.5" rot="R90"/>
 <instance part="C2" gate="G$1" x="132.08" y="94.615" rot="R90"/>
+<instance part="USB" gate="G$1" x="146.05" y="19.685"/>
 </instances>
 <busses>
@@
 </segment>
 <segment>
-<wire x1="141.986" y1="18.415" x2="162.052" y2="18.415" width="0.1524" layer="91"/>
-<label x="142.24" y="16.51" size="1.778" layer="95"/>
+<wire x1="115.951" y1="14.605" x2="138.43" y2="14.605" width="0.1524" layer="91"/>
+<label x="116.205" y="15.24" size="1.778" layer="95"/>
 <pinref part="USB" gate="G$1" pin="GND"/>
+<wire x1="138.43" y1="14.605" x2="138.43" y2="6.985" width="0.1524" layer="91"/>
+<wire x1="138.43" y1="6.985" x2="167.005" y2="6.985" width="0.1524" layer="91"/>
+<junction x="138.43" y="14.605"/>
+<pinref part="USB" gate="G$1" pin="SHIELD"/>
+<wire x1="153.67" y1="19.685" x2="167.005" y2="19.685" width="0.1524" layer="91"/>
+<wire x1="167.005" y1="19.685" x2="167.005" y2="6.985" width="0.1524" layer="91"/>
 </segment>
 </net>
@@
 </segment>
 <segment>
-<wire x1="141.986" y1="20.955" x2="162.052" y2="20.955" width="0.1524" layer="91"/>
-<label x="142.24" y="20.955" size="1.778" layer="95"/>
-<pinref part="USB" gate="G$1" pin="VBUS"/>
+<wire x1="115.951" y1="24.765" x2="138.43" y2="24.765" width="0.1524" layer="91"/>
+<label x="116.205" y="25.4" size="1.778" layer="95"/>
+<pinref part="USB" gate="G$1" pin="VCC"/>
 </segment>
 </net>
@@
 </sheet>
 </sheets>
+<errors>
+</errors>
 </schematic>
 </drawing>
