File: ESP8266_MySensorsGateway/ESP8266_MySensorsGateway_v1.3.brd (EAGLE design)
At the start: 50 x 24.9 mm, 38 parts, among them IC1 3V3

Commit message: version 1.3
Parts:
- USB: value USB-MICROB -> USB_MICROB_PLUGCONN-11752; device SparkFun-Connectors:USB-MICROB -> SparkFun-Connectors:USB-B-MICRO-SMD_V03
- moved D1 0.68 mm to (7.05, 66.5)
- moved U$2 0.40 mm to (7.04, 51.4)
- moved USB 0.31 mm to (3.23, 68.1), turned to 180 degrees
- flipped PRG to the bottom, turned to 180 degrees
Connections:
- net GND: now also USB.GND1, USB.SHIELD1, USB.SHIELD2, USB.SHIELD3; no longer USB.GND, USB.MT1, USB.MT2
- net VUSB: now also USB.VBUS1; no longer USB.VBUS
Routing:
- net GND: track 96.1 -> 85.1 mm, vias 16 -> 21
- net VUSB: track 8.10 -> 7.08 mm
- net VIN: track 5.13 -> 4.56 mm
- net N$10: track 15.7 -> 15.1 mm
Other:
- board text added: "ESP/MS-GW/v1.3/21.02.2016"
- board text added: "PRG"
- board text removed: "ESP/MS-GW/v1.3/13.02.2016"

Commit message: kleinere optimierungen
Parts:
- moved FLASH 0.89 mm to (25.9, 57.5)
- moved RST 0.89 mm to (25.9, 53.7)
Routing:
- net GND: track 85.1 -> 83.2 mm, vias 21 -> 20
- net N$7: track 3.81 -> 5.40 mm
- net VCC: track 100.6 -> 102.1 mm
- net GPIO0: track 43.4 -> 42.2 mm
- net LED_ERR: track 38.9 -> 39.9 mm
- net RXD: track 52.4 -> 53.4 mm
- net RST: track 49.7 -> 48.8 mm

Commit message: .
Routing:
- net VCC: track 102.1 -> 103.6 mm
- net RXD: track 53.4 -> 54.6 mm
- net LED_ERR: track 39.9 -> 40.8 mm
- net GND: track 83.2 -> 84.0 mm
- net TXD: track 56.0 -> 56.6 mm
- net SCK: track 33.5 -> 34.1 mm
