File: ESP8266_MySensorsGateway/ESP8266_MySensorsGateway_v1.4.1.sch (EAGLE design)
At the start: 37 parts, among them IC1 3V3, IC4 ATSHA204A

Commit message: .
Parts:
- added SJ2, SJ3: JUMPER-PAD-3-NOYES_SILK, SparkFun-Passives:JUMPER-PAD-3-NOYES_SILK
Connections:
- new net D3: ESP.GPIO0, R15.2, R5.1, SJ2.3, SJ3.1
- new net D4: ESP.GPIO2, R4.1, SJ2.1, SJ3.3
- net ATSHA: now also SJ2.2; no longer ESP.GPIO0, R15.2, R5.1
- net LED_ERR: now also SJ3.2; no longer ESP.GPIO2, R4.1
Other:
- note added: "D3"
- note added: "D4"
- note removed: "(D3)"
- moved on the sheet: IC4, INCLUSION
Changed lines of the file:
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@@
 <part name="IC4" library="Sensor" deviceset="ATSHA204A" device=""/>
 <part name="GND4" library="supply1" deviceset="GND" device=""/>
+<part name="SJ2" library="SparkFun-Passives" deviceset="JUMPER-PAD-3-NO" device="YES_SILK"/>
+<part name="SJ3" library="SparkFun-Passives" deviceset="JUMPER-PAD-3-NO" device="YES_SILK"/>
 </parts>
 <sheets>
@@
 <text x="-13.97" y="-19.05" size="1.778" layer="97">TX (Y)</text>
 <text x="-22.86" y="-27.94" size="1.778" layer="97">RX (G)</text>
-<text x="53.34" y="20.32" size="1.778" layer="97">(D3)</text>
+<text x="53.975" y="20.32" size="1.778" layer="97">D3</text>
+<text x="59.055" y="20.32" size="1.778" layer="97">D4</text>
 </plain>
 <instances>
@@
 <instance part="P+1" gate="VCC" x="123.825" y="55.245" rot="R90"/>
 <instance part="GND1" gate="1" x="120.015" y="57.785" rot="R270"/>
-<instance part="INCLUSION" gate="G$1" x="26.67" y="-26.035" rot="R270"/>
-<instance part="GND2" gate="1" x="42.545" y="-26.035" rot="R90"/>
+<instance part="INCLUSION" gate="G$1" x="20.32" y="-26.67" rot="R270"/>
+<instance part="GND2" gate="1" x="36.195" y="-26.67" rot="R90"/>
 <instance part="R12" gate="G$1" x="-50.165" y="-8.89"/>
 <instance part="R13" gate="G$1" x="-50.165" y="-17.78"/>
@@
 <instance part="C2" gate="G$1" x="132.08" y="94.615" rot="R90"/>
 <instance part="USB" gate="G$1" x="146.05" y="19.685"/>
-<instance part="IC4" gate="U1" x="24.765" y="-1.27"/>
-<instance part="GND4" gate="1" x="9.525" y="-1.27" rot="R270"/>
+<instance part="IC4" gate="U1" x="18.415" y="-1.905"/>
+<instance part="GND4" gate="1" x="3.175" y="-1.905" rot="R270"/>
+<instance part="SJ2" gate="G$1" x="50.165" y="-13.97" smashed="yes" rot="MR180"/>
+<instance part="SJ3" gate="G$1" x="60.325" y="-13.97" smashed="yes" rot="MR0"/>
 </instances>
 <busses>
@@
 </segment>
 <segment>
-<label x="37.465" y="1.905" size="1.778" layer="95"/>
+<label x="31.115" y="1.27" size="1.778" layer="95"/>
 <pinref part="IC4" gate="U1" pin="VCC"/>
-<wire x1="34.925" y1="1.27" x2="40.64" y2="1.27" width="0.1524" layer="91"/>
+<wire x1="28.575" y1="0.635" x2="34.29" y2="0.635" width="0.1524" layer="91"/>
 </segment>
 </net>
@@
 <pinref part="INCLUSION" gate="G$1" pin="2"/>
 <pinref part="GND2" gate="1" pin="GND"/>
-<wire x1="40.005" y1="-26.035" x2="31.75" y2="-26.035" width="0.1524" layer="91"/>
+<wire x1="33.655" y1="-26.67" x2="25.4" y2="-26.67" width="0.1524" layer="91"/>
 </segment>
 <segment>
@@
 <segment>
 <pinref part="IC4" gate="U1" pin="GND"/>
-<wire x1="14.605" y1="-1.27" x2="12.065" y2="-1.27" width="0.1524" layer="91"/>
+<wire x1="8.255" y1="-1.905" x2="5.715" y2="-1.905" width="0.1524" layer="91"/>
 <pinref part="GND4" gate="1" pin="GND"/>
 </segment>
@@
 </segment>
 <segment>
-<pinref part="ESP" gate="G$1" pin="GPIO2"/>
-<wire x1="30.48" y1="76.2" x2="60.96" y2="76.2" width="0.1524" layer="91"/>
-<pinref part="R4" gate="G$1" pin="1"/>
-<wire x1="60.96" y1="76.2" x2="60.96" y2="106.68" width="0.1524" layer="91"/>
-<junction x="60.96" y="76.2"/>
-<wire x1="60.96" y1="76.2" x2="60.96" y2="19.05" width="0.1524" layer="91"/>
-<label x="60.96" y="24.13" size="1.778" layer="95" rot="R90"/>
+<pinref part="SJ3" gate="G$1" pin="2"/>
+<wire x1="65.405" y1="-13.97" x2="69.215" y2="-13.97" width="0.1524" layer="91"/>
+<label x="67.31" y="-13.335" size="1.778" layer="95"/>
 </segment>
 </net>
 <net name="INCL" class="0">
 <segment>
-<label x="6.35" y="-26.035" size="1.778" layer="95"/>
+<label x="0" y="-26.67" size="1.778" layer="95"/>
 <pinref part="INCLUSION" gate="G$1" pin="1"/>
-<wire x1="21.59" y1="-26.035" x2="5.08" y2="-26.035" width="0.1524" layer="91"/>
+<wire x1="15.24" y1="-26.67" x2="-1.27" y2="-26.67" width="0.1524" layer="91"/>
 </segment>
 <segment>
@@
 <net name="ATSHA" class="0">
 <segment>
-<wire x1="34.925" y1="-3.81" x2="40.64" y2="-3.81" width="0.1524" layer="91"/>
-<label x="37.465" y="-3.175" size="1.778" layer="95"/>
+<wire x1="28.575" y1="-4.445" x2="34.29" y2="-4.445" width="0.1524" layer="91"/>
+<label x="31.115" y="-3.81" size="1.778" layer="95"/>
 <pinref part="IC4" gate="U1" pin="SDA"/>
+</segment>
+<segment>
+<pinref part="SJ2" gate="G$1" pin="2"/>
+<wire x1="45.085" y1="-13.97" x2="40.64" y2="-13.97" width="0.1524" layer="91"/>
+<label x="39.37" y="-13.335" size="1.778" layer="95"/>
+</segment>
+</net>
+<net name="D3" class="0">
+<segment>
+<pinref part="SJ2" gate="G$1" pin="3"/>
+<wire x1="50.165" y1="-8.89" x2="50.165" y2="-6.985" width="0.1524" layer="91"/>
+<pinref part="SJ3" gate="G$1" pin="1"/>
+<wire x1="50.165" y1="-6.985" x2="58.42" y2="-6.985" width="0.1524" layer="91"/>
+<wire x1="58.42" y1="-6.985" x2="60.325" y2="-6.985" width="0.1524" layer="91"/>
+<wire x1="60.325" y1="-6.985" x2="60.325" y2="-8.89" width="0.1524" layer="91"/>
+<label x="55.88" y="-5.08" size="1.778" layer="95" rot="R180"/>
+<wire x1="58.42" y1="-6.985" x2="58.42" y2="-3.81" width="0.1524" layer="91"/>
+<junction x="58.42" y="-6.985"/>
 </segment>
 <segment>
@@
 <wire x1="69.85" y1="78.74" x2="55.88" y2="78.74" width="0.1524" layer="91"/>
 <wire x1="55.88" y1="78.74" x2="30.48" y2="78.74" width="0.1524" layer="91"/>
-<wire x1="55.88" y1="78.74" x2="55.88" y2="25.4" width="0.1524" layer="91"/>
+<wire x1="55.88" y1="78.74" x2="55.88" y2="22.86" width="0.1524" layer="91"/>
 <junction x="55.88" y="78.74"/>
 <label x="55.88" y="25.4" size="1.778" layer="95" rot="R90"/>
@@
 </segment>
 </net>
+<net name="D4" class="0">
+<segment>
+<pinref part="SJ3" gate="G$1" pin="3"/>
+<wire x1="60.325" y1="-19.05" x2="60.325" y2="-20.32" width="0.1524" layer="91"/>
+<pinref part="SJ2" gate="G$1" pin="1"/>
+<wire x1="60.325" y1="-20.32" x2="58.42" y2="-20.32" width="0.1524" layer="91"/>
+<wire x1="58.42" y1="-20.32" x2="50.165" y2="-20.32" width="0.1524" layer="91"/>
+<wire x1="50.165" y1="-20.32" x2="50.165" y2="-19.05" width="0.1524" layer="91"/>
+<label x="55.88" y="-20.955" size="1.778" layer="95" rot="R180"/>
+<wire x1="58.42" y1="-20.32" x2="58.42" y2="-23.495" width="0.1524" layer="91"/>
+<junction x="58.42" y="-20.32"/>
+</segment>
+<segment>
+<pinref part="ESP" gate="G$1" pin="GPIO2"/>
+<wire x1="30.48" y1="76.2" x2="60.96" y2="76.2" width="0.1524" layer="91"/>
+<pinref part="R4" gate="G$1" pin="1"/>
+<wire x1="60.96" y1="76.2" x2="60.96" y2="106.68" width="0.1524" layer="91"/>
+<junction x="60.96" y="76.2"/>
+<wire x1="60.96" y1="76.2" x2="60.96" y2="22.86" width="0.1524" layer="91"/>
+<label x="60.96" y="24.13" size="1.778" layer="95" rot="R90"/>
+</segment>
+</net>
