File: ESP8266_1wire_Gateway_WeMosD1Mini/ESP8266_1wire_Gateway_NodeMCU_WeMosD1Mini_max.brd (EAGLE design)
At the start: 124.3 x 50 mm, 58 parts, among them IC1 7805, IC2 5V, IC3 DS2482-100S, IC4 DS18B20, M1 WEMOS, Q1 BSS84, Q2 BSS138, Q3 BSS138, Q4 BSS138

Commit message: version 1.0
Parts:
- C1: value 470p -> 470p*
- R1: value pullup* -> 1k-2k2*
- SJ2: value bypass l.shift -> bypass
- SJ3: value 1w-VCC: 5V | 3V3 -> 5V | 3V3
- SJ4: value Direkt | BusMaster -> direct | busmaster
- moved U$2 33.5 mm to (44.4, 67.8)
- moved U$1 0.63 mm to (13.3, 71.0)
Routing:
- net GND: vias 6 -> 20
Other:
- board size 124.3 x 50 mm -> 49.5 x 49.5 mm
- board text added: "1w power"
- board text added: "1w pullup"
- board text added: "1wire"
- board text added: "1wire bus"
- board text added: "ESD"
- board text added: "ESP 1wire Gateway R1.0 / 25.06.16"
- board text added: "ESP-1w-Gateway R1.0 / 25.06.16 s6z.de"
- board text added: "GND*"
- board text added: "Power"
- board text added: "SJ1"
- board text added: "SJ2"
- board text added: "SJ3"
- board text added: "SJ4"
- board text added: "Stromversorgung: =>5V: SJ1 geschlossen, IC1, IC2 (C3, C4) unbestueckt =>7-12V: SJ1 offen, IC2 bestueckt (1117 5.0), C3, C4 bestueckt, IC1 unbestueckt =>13-24V: SJ1 offen, IC2 unbestueckt, IC1 bestueckt (7805), C3, C4 bestueckt. Bus Konfiguration: generell: - SJ3 regelt die Stromversorgung des Busses (gilt nicht für parasitaer versorgte Devices). - ZD1 (ESD protection) kann überbrueckt werden - R1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"
- board text added: "VCC*"
- board text added: "bus master"
- board text added: "filter"
- board text added: "level shifter (1w direct)"
- board text added: "level shifter (i2c)"
- board text added: "s6z.de"
- board text added: "strong pullup"
- board text removed: "1W VCC"
- board text removed: "ESP-1w_GW R0.9 / 24.06.16"
- board text removed: "Power in: 5V: SJ1 geschlossen, IC1, IC2 (C3, C4) unbestückt 7-12V: SJ1 offen, IC2 bestückt (1117), C3,C4 bestückt, IC1 unbestückt 13-24V: SJ1 offen, IC2 unbestückt, IC1 bestückt (7805), C3, C4 bestückt. onewire: genrell: SJ3 soll eine korrekte Einstellung je nach Betriebsart 3,3V/5V aufweisen ZD1 (ESD protetion) kann überbrückt werden R17 und C1 bilden einen optionale Filter. R17 ist jedoch meist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"
