File: ESP8266_1wire_Gateway_WeMosD1Mini/ESP8266_1wire_Gateway_NodeMCU_WeMosD1Mini_max.brd (EAGLE design)
At the start: 49.5 x 49.5 mm, 58 parts, among them IC1 7805, IC2 5V, IC3 DS2482-100S, IC4 DS18B20, M1 WEMOS, Q1 BSS84, Q2 BSS138, Q3 BSS138, Q4 BSS138

Commit message: v1.2
Parts:
- R18: value cur.limit -> cur.limit (50-100)
- turned LED1 to 90 degrees
Connections:
- net GND: now also LED1.C; no longer LED1.A
- net N$4: now also LED1.A; no longer LED1.C
Routing:
- net GND: track 215.3 -> 214.8 mm
Other:
- board text added: "ESP 1wire Gateway R1.2 / 04.09.16"
- board text added: "ESP-1w-Gateway R1.2 / 04.09.16 s6z.de"
- board text removed: "ESP 1wire Gateway R1.1 / 24.08.16"
- board text removed: "ESP-1w-Gateway R1.1 / 24.08.16 s6z.de"

Commit message: v1.3 (new diode to protect ams1117 by power over usb)
Parts:
- added D2: SS14, ihpcb-diode:DO214
- moved PF1 4.08 mm to (23.1, 39.3)
- moved IC2 0.30 mm to (14.6, 33.6)
Connections:
- new net 5V_WEMOS: D2.CATHODE, M1.5V, PF1.2
- net 5V_IN: now also D2.ANODE; no longer M1.5V, PF1.2
Routing:
- net 5V_WEMOS: track 0.00 -> 46.5 mm
- net 5V_IN: track 74.7 -> 28.6 mm
- net VCC_5V: track 154.1 -> 153.2 mm
Other:
- board text added: "ESP 1wire Gateway R1.3 / 05.09.16"
- board text added: "ESP-1w-Gateway R1.3 / 05.09.16 s6z.de"
- board text removed: "ESP 1wire Gateway R1.2 / 04.09.16"
- board text removed: "ESP-1w-Gateway R1.2 / 04.09.16 s6z.de"

Commit message: Schutzdiode + Korrekturen
Parts:
- added R5: 470, resistor:R0805
- moved SJ1 2.16 mm to (14.6, 27.7), turned to 180 degrees
Connections:
- net GPIO16_WAKE: now also R5.2
- net N$8: no longer SJ1.1
- net RST: now also R5.1
- net VIN: now also SJ1.1
Routing:
- net VIN: track 7.53 -> 18.8 mm, vias 1 -> 2
- net RST: track 32.1 -> 41.9 mm
- net GPIO16_WAKE: track 0.00 -> 6.33 mm
- net 1W_BUSM: track 27.7 -> 32.9 mm
- net 5V_IN: track 28.6 -> 27.2 mm
- net N$8: track 21.8 -> 20.7 mm
- net GND: track 214.6 -> 214.7 mm, vias 20 -> 17
Other:
- board text added: "ESP 1wire Gateway R1.5 / 07.09.16"
- board text added: "ESP-1w-Gateway R1.5 / 07.09.16 s6z.de"
- board text added: "wakeup"
- board text removed: "ESP 1wire Gateway R1.3 / 05.09.16"
- board text removed: "ESP-1w-Gateway R1.3 / 05.09.16 s6z.de"
